Commit message: ...

File: m2wr_robot/urdf/caster.xacro (robot description, xacro)
@@ -36,7 +36,7 @@
             </collision>
         </link>
-        <gazebo reference="${prefix}_link">
-            <material>Gazebo/Gray</material>
-        </gazebo>
+        <!--<gazebo reference="${prefix}_link">-->
+            <!--<material>Gazebo/Gray</material>-->
+        <!--</gazebo>-->
     </xacro:macro>
 </robot>

File: m2wr_robot/urdf/m2wr.xacro (robot description, xacro)
@@ -5,11 +5,5 @@
     <xacro:include filename="$(find m2wr_robot)/urdf/wheel.xacro" />
     <xacro:include filename="$(find m2wr_robot)/urdf/caster.xacro" />
-    <!-- materials -->
-    <material name="gray">
-        <color rgba="0.5 0.5 0.5 2.5"/>
-    </material>
-    <material name="red">
-        <color rgba="1.0 0.0 0.0 2.5"/>
-    </material>
+    <xacro:include filename="$(find m2wr_robot)/urdf/materials.xacro" />
     <!-- base -->
     <link name="base_link"/>
@@ -41,7 +35,7 @@
         </collision>
     </link>
-    <gazebo reference="body_link">
-        <material>Gazebo/Gray</material>
-    </gazebo>
+    <!--<gazebo reference="body_link">-->
+        <!--<material>Gazebo/Gray</material>-->
+    <!--</gazebo>-->
     <!-- front and back caster -->
     <xacro:caster_macro prefix="front_caster" parent="base_link" xyz="0.08 0 0.04" r="0.04"/>

File: m2wr_robot/urdf/wheel.xacro (robot description, xacro)
@@ -28,7 +28,7 @@
             </collision>
         </link>
-        <gazebo reference="${prefix}_link">
-          <material>Gazebo/Red</material>
-        </gazebo>
+        <!--<gazebo reference="${prefix}_link">-->
+          <!--<material>Gazebo/Red</material>-->
+        <!--</gazebo>-->
     </xacro:macro>
 </robot>

Commit message: ...

File: m2wr_robot/urdf/caster.xacro (robot description, xacro)
@@ -1,4 +1,4 @@
 <?xml version="1.0"?>
-<robot xmlns:xacro="http://www.ros.org/wiki/xacro">
+<robot xmlns:xacro="http://ros.org/wiki/xacro">
     <xacro:macro name="caster_macro" params="parent prefix xyz r">
         <!-- joint -->
@@ -36,7 +36,7 @@
             </collision>
         </link>
-        <!--<gazebo reference="${prefix}_link">-->
-            <!--<material>Gazebo/Gray</material>-->
-        <!--</gazebo>-->
+        <gazebo reference="${prefix}_link">
+            <material>Gazebo/Gray</material>
+        </gazebo>
     </xacro:macro>
 </robot>

File: m2wr_robot/urdf/m2wr.xacro (robot description, xacro)
@@ -35,7 +35,7 @@
         </collision>
     </link>
-    <!--<gazebo reference="body_link">-->
-        <!--<material>Gazebo/Gray</material>-->
-    <!--</gazebo>-->
+    <gazebo reference="body_link">
+        <material>Gazebo/Gray</material>
+    </gazebo>
     <!-- front and back caster -->
     <xacro:caster_macro prefix="front_caster" parent="base_link" xyz="0.08 0 0.04" r="0.04"/>

File: m2wr_robot/urdf/materials.xacro (robot description, xacro)
@@ -1,4 +1,4 @@
 <?xml version="1.0"?>
-<robot xmlns:xacro="http://www.ros.org/wiki/xacro">
+<robot xmlns:xacro="http://ros.org/wiki/xacro">
   <material name="black">
     <color rgba="0.0 0.0 0.0 1.0"/>

File: m2wr_robot/urdf/wheel.xacro (robot description, xacro)
@@ -1,4 +1,4 @@
 <?xml version="1.0"?>
-<robot xmlns:xacro="http://www.ros.org/wiki/xacro">
+<robot xmlns:xacro="http://ros.org/wiki/xacro">
     <xacro:macro name="wheel_macro" params="parent prefix xyz">
         <!-- joint -->
@@ -28,7 +28,7 @@
             </collision>
         </link>
-        <!--<gazebo reference="${prefix}_link">-->
-          <!--<material>Gazebo/Red</material>-->
-        <!--</gazebo>-->
+        <gazebo reference="${prefix}_link">
+          <material>Gazebo/Red</material>
+        </gazebo>
     </xacro:macro>
 </robot>

Commit message: ...

File: m2wr_robot/urdf/caster.xacro (robot description, xacro)
@@ -18,5 +18,5 @@
             </visual>
             <collision>
-                <!--<origin xyz="0 0 0" rpy="0 0 0" />-->
+                <origin xyz="0 0 0" rpy="0 0 0" />
                 <geometry>
                     <sphere radius="${r}" />

Commit message: ...

File: m2wr_robot/urdf/caster.xacro (robot description, xacro)
@@ -2,10 +2,4 @@
 <robot xmlns:xacro="http://ros.org/wiki/xacro">
     <xacro:macro name="caster_macro" params="parent prefix xyz r">
-        <!-- joint -->
-        <joint name="${prefix}_joint" type="fixed">
-            <parent link="${parent}"/>
-            <child  link="${prefix}_link"/>
-            <origin xyz="${xyz}" rpy="0 0 0"/>
-        </joint>
         <!-- link -->
         <link name="${prefix}_link">

File: m2wr_robot/urdf/m2wr.xacro (robot description, xacro)
@@ -39,6 +39,6 @@
     </gazebo>
     <!-- front and back caster -->
-    <xacro:caster_macro prefix="front_caster" parent="base_link" xyz="0.08 0 0.03" r="0.04"/>
-    <xacro:caster_macro prefix="back_caster" parent="base_link" xyz="-0.08 0 0.03" r="0.04"/>
+    <xacro:caster_macro prefix="front_caster" parent="base_link" xyz="0.08 0 0.04" r="0.04"/>
+    <xacro:caster_macro prefix="back_caster" parent="base_link" xyz="-0.08 0 0.04" r="0.04"/>
     <!-- left and right wheel -->
     <xacro:wheel_macro prefix="left_wheel"  parent="base_link" xyz="0 0.1 0.05"/>

Commit message: ...

File: m2wr_robot/urdf/caster.xacro (robot description, xacro)
@@ -2,4 +2,10 @@
 <robot xmlns:xacro="http://ros.org/wiki/xacro">
     <xacro:macro name="caster_macro" params="parent prefix xyz r">
+        <!-- joint -->
+        <joint name="${prefix}_joint" type="fixed">
+            <parent link="${parent}"/>
+            <child  link="${prefix}_link"/>
+            <origin xyz="${xyz}" rpy="0 0 0"/>
+        </joint>
         <!-- link -->
         <link name="${prefix}_link">

File: m2wr_robot/urdf/m2wr.xacro (robot description, xacro)
@@ -38,4 +38,54 @@
         <material>Gazebo/Gray</material>
     </gazebo>
+    <visual>
+        <origin xyz="0.08 0 0.04" rpy="0 0 0" />
+        <geometry>
+            <sphere radius="0.04" />
+        </geometry>
+        <material name="gray" />
+    </visual>
+    <collision>
+        <origin xyz="0.08 0 0.04" rpy="0 0 0" />
+        <geometry>
+            <sphere radius="0.04" />
+        </geometry>
+        <surface>
+            <friction>
+                <!-- frictionless between these two surface -->
+                <ode>
+                    <mu>0</mu>
+                    <mu2>0</mu2>
+                    <slip1>1.0</slip1>
+                    <slip2>1.0</slip2>
+                </ode>
+            </friction>
+        </surface>
+        <material name="gray" />
+    </collision>
+    <visual>
+        <origin xyz="-0.08 0 0.04" rpy="0 0 0" />
+        <geometry>
+            <sphere radius="0.04" />
+        </geometry>
+        <material name="gray" />
+    </visual>
+    <collision>
+        <origin xyz="-0.08 0 0.04" rpy="0 0 0" />
+        <geometry>
+            <sphere radius="0.04" />
+        </geometry>
+        <surface>
+            <friction>
+                <!-- frictionless between these two surface -->
+                <ode>
+                    <mu>0</mu>
+                    <mu2>0</mu2>
+                    <slip1>1.0</slip1>
+                    <slip2>1.0</slip2>
+                </ode>
+            </friction>
+        </surface>
+        <material name="gray" />
+    </collision>
     <!-- front and back caster -->
     <xacro:caster_macro prefix="front_caster" parent="base_link" xyz="0.08 0 0.04" r="0.04"/>

Commit message: ...

File: m2wr_robot/urdf/caster.xacro (robot description, xacro)
@@ -22,15 +22,4 @@
                     <sphere radius="${r}" />
                 </geometry>
-                <surface>
-                    <friction>
-                        <!-- frictionless between these two surface -->
-                        <ode>
-                            <mu>0</mu>
-                            <mu2>0</mu2>
-                            <slip1>1.0</slip1>
-                            <slip2>1.0</slip2>
-                        </ode>
-                    </friction>
-                </surface>
                 <material name="gray" />
             </collision>
@@ -38,4 +27,6 @@
         <gazebo reference="${prefix}_link">
             <material>Gazebo/Gray</material>
+            <mu1 value="0.5" />
+            <mu2 value="0.5" />
         </gazebo>
     </xacro:macro>

File: m2wr_robot/urdf/m2wr.xacro (robot description, xacro)
@@ -2,20 +2,26 @@
 <robot name="m2wr" xmlns:xacro="http://ros.org/wiki/xacro">
     <!-- inludes -->
-    <xacro:include filename="$(find m2wr_robot)/urdf/car_driver.gazebo" />
+    <!--<xacro:include filename="$(find m2wr_robot)/urdf/car_driver.gazebo" />-->
     <xacro:include filename="$(find m2wr_robot)/urdf/wheel.xacro" />
-    <!--<xacro:include filename="$(find m2wr_robot)/urdf/caster.xacro" />-->
+    <xacro:include filename="$(find m2wr_robot)/urdf/caster.xacro" />
     <xacro:include filename="$(find m2wr_robot)/urdf/materials.xacro" />
-    <!-- base -->
-    <link name="base_link">
-        <pose>0 0 0 0 0 0</pose>
+    <link name="base_link"/>
+    <!-- body : joint -->
+    <joint name="body_joint" type="fixed">
+        <parent link="base_link"/>
+        <child  link="body_link"/>
+        <origin xyz="-0.07 0 0.07" rpy="0 0 0"/>
+    </joint>
+    <!-- body : link -->
+    <link name="body_link">
         <inertial>
             <origin xyz="0 0 0" rpy="0 0 0"/>
-            <mass value="5.0"/>
-            <inertia ixx="0.04" ixy="0.0" ixz="0.0" iyy="0.1" iyz="0.0" izz="0.1"/>
+            <mass value="1.0"/>
+            <inertia ixx="0.001" ixy="0.0" ixz="0.0" iyy="0.001" iyz="0.0" izz="0.001"/>
         </inertial>
         <visual>
             <origin xyz="0 0 0" rpy="0 0 0" />
             <geometry>
-                <box size="0.5 0.3 0.07" />
+                <box size="0.24 0.18 0.06" />
             </geometry>
             <material name="gray" />
@@ -24,64 +30,17 @@
             <origin xyz="0 0 0" rpy="0 0 0" />
             <geometry>
-                <box size="0.5 0.3 0.07" />
+                <box size="0.24 0.178 0.06" />
             </geometry>
         </collision>
-        <!-- caster front -->
-        <collision name="caster_front_collision">
-            <origin rpy=" 0 0 0" xyz="0.35 0 -0.05"/>
-            <geometry>
-                <sphere radius="0.05"/>
-            </geometry>
-            <surface>
-                <friction>
-                    <!-- frictionless between these two surface -->
-                    <ode>
-                        <mu>0</mu>
-                        <mu2>0</mu2>
-                        <slip1>1.0</slip1>
-                        <slip2>1.0</slip2>
-                    </ode>
-                </friction>
-            </surface>
-        </collision>
-        <visual name="caster_front_visual">
-            <origin rpy=" 0 0 0" xyz="0.2 0 -0.05"/>
-            <geometry>
-                <sphere radius="0.05"/>
-            </geometry>
-        </visual>
-        <!-- caster back -->
-        <collision name="caster_back_collision">
-            <origin rpy=" 0 0 0" xyz="-0.35 0 -0.05"/>
-            <geometry>
-                <sphere radius="0.05"/>
-            </geometry>
-            <surface>
-                <friction>
-                    <!-- frictionless between these two surface -->
-                    <ode>
-                        <mu>0</mu>
-                        <mu2>0</mu2>
-                        <slip1>1.0</slip1>
-                        <slip2>1.0</slip2>
-                    </ode>
-                </friction>
-            </surface>
-        </collision>
-        <visual name="caster_back_visual">
-            <origin rpy=" 0 0 0" xyz="-0.2 0 -0.05"/>
-            <geometry>
-                <sphere radius="0.05"/>
-            </geometry>
-        </visual>
     </link>
-    <gazebo reference="base_link">
+    <gazebo reference="body_link">
         <material>Gazebo/Gray</material>
     </gazebo>
+    <xacro:caster_macro prefix="caster" parent="base_link" xyz="-0.14 0 0.04" r="0.04"/>
     <!-- front and back caster -->
-    <!--<xacro:caster_macro prefix="front_caster" parent="base_link" xyz="0.08 0 0.04" r="0.04"/>-->
+    <!--<<xacro:caster_macro prefix="front_caster" parent="base_link" xyz="0.08 0 0.04" r="0.04"/>-->
     <!--<xacro:caster_macro prefix="back_caster" parent="base_link" xyz="-0.08 0 0.04" r="0.04"/>-->
     <!-- left and right wheel -->
-    <xacro:wheel_macro prefix="left_wheel"  parent="base_link" xyz="0 0.2 0.0"/>
-    <xacro:wheel_macro prefix="right_wheel" parent="base_link" xyz="0 -0.2 0.0"/>
+    <xacro:wheel_macro prefix="left_wheel"  parent="base_link" xyz="0  0.1 0.05" r="0.05"/>
+    <xacro:wheel_macro prefix="right_wheel" parent="base_link" xyz="0 -0.1 0.05" r="0.05"/>
 </robot>

File: m2wr_robot/urdf/wheel.xacro (robot description, xacro)
@@ -1,5 +1,5 @@
 <?xml version="1.0"?>
 <robot xmlns:xacro="http://ros.org/wiki/xacro">
-    <xacro:macro name="wheel_macro" params="parent prefix xyz">
+    <xacro:macro name="wheel_macro" params="parent prefix xyz r">
         <!-- joint -->
         <joint name="${prefix}_joint" type="continuous">
@@ -18,5 +18,5 @@
             <visual>
                 <geometry>
-                    <cylinder radius="0.05" length="0.02" />
+                    <cylinder radius="${r}" length="0.02" />
                 </geometry>
                 <material name="red"/>
@@ -24,5 +24,5 @@
             <collision>
                 <geometry>
-                    <cylinder radius="0.05" length="0.02" />
+                    <cylinder radius="${r}" length="0.02" />
                 </geometry>
             </collision>
