Commit message: ...

File: m2wr_robot/urdf/m2wr0.xacro (robot description, xacro)
@@ -2,7 +2,7 @@
 <robot name="m2wr" xmlns:xacro="http://ros.org/wiki/xacro">
     <!-- inludes -->
-    <!--<xacro:include filename="$(find m2wr_robot)/urdf/car_driver.gazebo" />-->
+    <xacro:include filename="$(find m2wr_robot)/urdf/car_driver.gazebo" />
     <xacro:include filename="$(find m2wr_robot)/urdf/wheel.xacro" />
-    <xacro:include filename="$(find m2wr_robot)/urdf/caster.xacro" />
+    <!--<xacro:include filename="$(find m2wr_robot)/urdf/caster.xacro" />-->
     <xacro:include filename="$(find m2wr_robot)/urdf/materials.xacro" />
     <link name="base_link"/>
@@ -37,5 +37,5 @@
         <material>Gazebo/Gray</material>
     </gazebo>
-    <xacro:caster_macro prefix="caster" parent="base_link" xyz="-0.14 0 0.04" r="0.04"/>
+    <!--<xacro:caster_macro prefix="caster" parent="base_link" xyz="-0.14 0 0.04" r="0.04"/>-->
     <!-- front and back caster -->
     <!--<<xacro:caster_macro prefix="front_caster" parent="base_link" xyz="0.08 0 0.04" r="0.04"/>-->
@@ -44,8 +44,3 @@
     <xacro:wheel_macro prefix="left_wheel"  parent="base_link" xyz="0  0.1 0.05" r="0.05"/>
     <xacro:wheel_macro prefix="right_wheel" parent="base_link" xyz="0 -0.1 0.05" r="0.05"/>
-    <gazebo>
-        <plugin name="gazebo_ros_control" filename="libgazebo_ros_control.so">
-            <robotNamespace>/m2wr</robotNamespace>
-        </plugin>
-    </gazebo>
 </robot>

File: m2wr_robot/urdf/wheel.xacro (robot description, xacro)
@@ -8,17 +8,5 @@
             <child  link="${prefix}_link"/>
             <axis xyz="0 0 1" />
-            <limit velocity="12.0" effort="0.4" />
-            <dynamics damping="0.1"/>
         </joint>
-        <!-- transimission -->
-        <transmission name="${prefix}_trans" type="SimpleTransmission">
-            <type>transmission_interface/SimpleTransmission</type>
-            <actuator name="${prefix}_motor">
-                <mechanicalReduction>1</mechanicalReduction>
-            </actuator>
-            <joint name="${prefix}_joint">
-                <hardwareInterface>hardware_interface/VelocityJointInterface</hardwareInterface>
-            </joint>
-        </transmission>
         <!-- link -->
         <link name="${prefix}_link">
@@ -42,9 +30,4 @@
         <gazebo reference="${prefix}_link">
             <material>Gazebo/Red</material>
-            <material>Gazebo/Red</material>
-            <mu1 value="2.5" />
-            <mu2 value="2.5" />
-            <kp value="50000" />
-            <kd value="10" />
         </gazebo>
     </xacro:macro>

Commit message: ...

File: m2wr_robot/urdf/m2wr0.xacro (robot description, xacro)
@@ -11,5 +11,5 @@
         <parent link="base_link"/>
         <child  link="body_link"/>
-        <origin xyz="-0.07 0 0.07" rpy="0 0 0"/>
+        <origin xyz="0 0 0.07" rpy="0 0 0"/>
     </joint>
     <!-- body : link -->
@@ -37,6 +37,6 @@
         <material>Gazebo/Gray</material>
     </gazebo>
-    <xacro:caster_macro prefix="back_caster" parent="base_link" xyz="-0.14 0 0.04" r="0.04"/>
-    <xacro:caster_macro prefix="front_caster" parent="base_link" xyz="0.14 0 0.04" r="0.04"/>
+    <xacro:caster_macro prefix="back_caster" parent="base_link" xyz="0.10 0 0.04" r="0.04"/>
+    <xacro:caster_macro prefix="front_caster" parent="base_link" xyz="0.10 0 0.04" r="0.04"/>
     <!-- front and back caster -->
     <!--<<xacro:caster_macro prefix="front_caster" parent="base_link" xyz="0.08 0 0.04" r="0.04"/>-->
