Commit message: ...

File: m2wr_robot/urdf/m2wr.xacro (robot description, xacro)
@@ -34,58 +34,58 @@
             </geometry>
         </collision>
+        <visual>
+            <origin xyz="0.08 0 0.04" rpy="0 0 0" />
+            <geometry>
+                <sphere radius="0.04" />
+            </geometry>
+            <material name="gray" />
+        </visual>
+        <collision>
+            <origin xyz="0.08 0 0.04" rpy="0 0 0" />
+            <geometry>
+                <sphere radius="0.04" />
+            </geometry>
+            <surface>
+                <friction>
+                    <!-- frictionless between these two surface -->
+                    <ode>
+                        <mu>0</mu>
+                        <mu2>0</mu2>
+                        <slip1>1.0</slip1>
+                        <slip2>1.0</slip2>
+                    </ode>
+                </friction>
+            </surface>
+            <material name="gray" />
+        </collision>
+        <visual>
+            <origin xyz="-0.08 0 0.04" rpy="0 0 0" />
+            <geometry>
+                <sphere radius="0.04" />
+            </geometry>
+            <material name="gray" />
+        </visual>
+        <collision>
+            <origin xyz="-0.08 0 0.04" rpy="0 0 0" />
+            <geometry>
+                <sphere radius="0.04" />
+            </geometry>
+            <surface>
+                <friction>
+                    <!-- frictionless between these two surface -->
+                    <ode>
+                        <mu>0</mu>
+                        <mu2>0</mu2>
+                        <slip1>1.0</slip1>
+                        <slip2>1.0</slip2>
+                    </ode>
+                </friction>
+            </surface>
+            <material name="gray" />
+        </collision>
     </link>
     <gazebo reference="body_link">
         <material>Gazebo/Gray</material>
     </gazebo>
-    <visual>
-        <origin xyz="0.08 0 0.04" rpy="0 0 0" />
-        <geometry>
-            <sphere radius="0.04" />
-        </geometry>
-        <material name="gray" />
-    </visual>
-    <collision>
-        <origin xyz="0.08 0 0.04" rpy="0 0 0" />
-        <geometry>
-            <sphere radius="0.04" />
-        </geometry>
-        <surface>
-            <friction>
-                <!-- frictionless between these two surface -->
-                <ode>
-                    <mu>0</mu>
-                    <mu2>0</mu2>
-                    <slip1>1.0</slip1>
-                    <slip2>1.0</slip2>
-                </ode>
-            </friction>
-        </surface>
-        <material name="gray" />
-    </collision>
-    <visual>
-        <origin xyz="-0.08 0 0.04" rpy="0 0 0" />
-        <geometry>
-            <sphere radius="0.04" />
-        </geometry>
-        <material name="gray" />
-    </visual>
-    <collision>
-        <origin xyz="-0.08 0 0.04" rpy="0 0 0" />
-        <geometry>
-            <sphere radius="0.04" />
-        </geometry>
-        <surface>
-            <friction>
-                <!-- frictionless between these two surface -->
-                <ode>
-                    <mu>0</mu>
-                    <mu2>0</mu2>
-                    <slip1>1.0</slip1>
-                    <slip2>1.0</slip2>
-                </ode>
-            </friction>
-        </surface>
-        <material name="gray" />
-    </collision>
     <!-- front and back caster -->
     <!--<xacro:caster_macro prefix="front_caster" parent="base_link" xyz="0.08 0 0.04" r="0.04"/>-->

Commit message: ...

File: m2wr_robot/urdf/m2wr.xacro (robot description, xacro)
@@ -35,5 +35,5 @@
         </collision>
         <visual>
-            <origin xyz="0.08 0 0.04" rpy="0 0 0" />
+            <origin xyz="0.08 0 0.03" rpy="0 0 0" />
             <geometry>
                 <sphere radius="0.04" />
@@ -42,5 +42,5 @@
         </visual>
         <collision>
-            <origin xyz="0.08 0 0.04" rpy="0 0 0" />
+            <origin xyz="0.08 0 0.03" rpy="0 0 0" />
             <geometry>
                 <sphere radius="0.04" />
@@ -60,5 +60,5 @@
         </collision>
         <visual>
-            <origin xyz="-0.08 0 0.04" rpy="0 0 0" />
+            <origin xyz="-0.08 0 0.03" rpy="0 0 0" />
             <geometry>
                 <sphere radius="0.04" />
@@ -67,5 +67,5 @@
         </visual>
         <collision>
-            <origin xyz="-0.08 0 0.04" rpy="0 0 0" />
+            <origin xyz="-0.08 0 0.03" rpy="0 0 0" />
             <geometry>
                 <sphere radius="0.04" />

Commit message: ...

File: m2wr_robot/urdf/m2wr.xacro (robot description, xacro)
@@ -4,25 +4,18 @@
     <xacro:include filename="$(find m2wr_robot)/urdf/car_driver.gazebo" />
     <xacro:include filename="$(find m2wr_robot)/urdf/wheel.xacro" />
-    <xacro:include filename="$(find m2wr_robot)/urdf/caster.xacro" />
+    <!--<xacro:include filename="$(find m2wr_robot)/urdf/caster.xacro" />-->
     <xacro:include filename="$(find m2wr_robot)/urdf/materials.xacro" />
     <!-- base -->
-    <link name="base_link"/>
-    <!-- body : joint -->
-    <joint name="body_joint" type="fixed">
-        <parent link="base_link"/>
-        <child  link="body_link"/>
-        <origin xyz="0 0 0.07" rpy="0 0 0"/>
-    </joint>
-    <!-- body : link -->
-    <link name="body_link">
+    <link name="base_link">
+        <pose>0 0 0 0 0 0</pose>
         <inertial>
             <origin xyz="0 0 0" rpy="0 0 0"/>
-            <mass value="1.0"/>
-            <inertia ixx="0.001" ixy="0.0" ixz="0.0" iyy="0.001" iyz="0.0" izz="0.001"/>
+            <mass value="5.0"/>
+            <inertia ixx="0.04" ixy="0.0" ixz="0.0" iyy="0.1" iyz="0.0" izz="0.1"/>
         </inertial>
         <visual>
             <!--<origin xyz="0 0 0" rpy="0 0 0" />-->
             <geometry>
-                <box size="0.24 0.18 0.06" />
+                <box size="0.5 0.3 0.07" />
             </geometry>
             <material name="gray" />
@@ -31,59 +24,9 @@
             <!--<origin xyz="0 0 0" rpy="0 0 0" />-->
             <geometry>
-                <box size="0.24 0.178 0.06" />
+                <box size="0.5 0.3 0.07" />
             </geometry>
         </collision>
-        <visual>
-            <origin xyz="0.08 0 0.03" rpy="0 0 0" />
-            <geometry>
-                <sphere radius="0.04" />
-            </geometry>
-            <material name="gray" />
-        </visual>
-        <collision>
-            <origin xyz="0.08 0 0.03" rpy="0 0 0" />
-            <geometry>
-                <sphere radius="0.04" />
-            </geometry>
-            <surface>
-                <friction>
-                    <!-- frictionless between these two surface -->
-                    <ode>
-                        <mu>0</mu>
-                        <mu2>0</mu2>
-                        <slip1>1.0</slip1>
-                        <slip2>1.0</slip2>
-                    </ode>
-                </friction>
-            </surface>
-            <material name="gray" />
-        </collision>
-        <visual>
-            <origin xyz="-0.08 0 0.03" rpy="0 0 0" />
-            <geometry>
-                <sphere radius="0.04" />
-            </geometry>
-            <material name="gray" />
-        </visual>
-        <collision>
-            <origin xyz="-0.08 0 0.03" rpy="0 0 0" />
-            <geometry>
-                <sphere radius="0.04" />
-            </geometry>
-            <surface>
-                <friction>
-                    <!-- frictionless between these two surface -->
-                    <ode>
-                        <mu>0</mu>
-                        <mu2>0</mu2>
-                        <slip1>1.0</slip1>
-                        <slip2>1.0</slip2>
-                    </ode>
-                </friction>
-            </surface>
-            <material name="gray" />
-        </collision>
     </link>
-    <gazebo reference="body_link">
+    <gazebo reference="base_link">
         <material>Gazebo/Gray</material>
     </gazebo>
@@ -92,5 +35,5 @@
     <!--<xacro:caster_macro prefix="back_caster" parent="base_link" xyz="-0.08 0 0.04" r="0.04"/>-->
     <!-- left and right wheel -->
-    <xacro:wheel_macro prefix="left_wheel"  parent="base_link" xyz="0 0.1 0.05"/>
-    <xacro:wheel_macro prefix="right_wheel" parent="base_link" xyz="0 -0.1 0.05"/>
+    <xacro:wheel_macro prefix="left_wheel"  parent="base_link" xyz="0 0.2 0.0"/>
+    <xacro:wheel_macro prefix="right_wheel" parent="base_link" xyz="0 -0.2 0.0"/>
 </robot>

Commit message: ...

File: m2wr_robot/urdf/m2wr.xacro (robot description, xacro)
@@ -27,4 +27,52 @@
             </geometry>
         </collision>
+        <!-- caster front -->
+        <collision name="caster_front_collision">
+            <origin rpy=" 0 0 0" xyz="0.35 0 -0.05"/>
+            <geometry>
+                <sphere radius="0.05"/>
+            </geometry>
+            <surface>
+                <friction>
+                    <!-- frictionless between these two surface -->
+                    <ode>
+                        <mu>0</mu>
+                        <mu2>0</mu2>
+                        <slip1>1.0</slip1>
+                        <slip2>1.0</slip2>
+                    </ode>
+                </friction>
+            </surface>
+        </collision>
+        <visual name="caster_front_visual">
+            <origin rpy=" 0 0 0" xyz="0.2 0 -0.05"/>
+            <geometry>
+                <sphere radius="0.05"/>
+            </geometry>
+        </visual>
+        <!-- caster back -->
+        <collision name="caster_back_collision">
+            <origin rpy=" 0 0 0" xyz="-0.35 0 -0.05"/>
+            <geometry>
+                <sphere radius="0.05"/>
+            </geometry>
+            <surface>
+                <friction>
+                    <!-- frictionless between these two surface -->
+                    <ode>
+                        <mu>0</mu>
+                        <mu2>0</mu2>
+                        <slip1>1.0</slip1>
+                        <slip2>1.0</slip2>
+                    </ode>
+                </friction>
+            </surface>
+        </collision>
+        <visual name="caster_back_visual">
+            <origin rpy=" 0 0 0" xyz="-0.2 0 -0.05"/>
+            <geometry>
+                <sphere radius="0.05"/>
+            </geometry>
+        </visual>
     </link>
     <gazebo reference="base_link">

Commit message: ...

File: m2wr_robot/urdf/m2wr.xacro (robot description, xacro)
@@ -15,5 +15,5 @@
         </inertial>
         <visual>
-            <!--<origin xyz="0 0 0" rpy="0 0 0" />-->
+            <origin xyz="0 0 0" rpy="0 0 0" />
             <geometry>
                 <box size="0.5 0.3 0.07" />
@@ -22,5 +22,5 @@
         </visual>
         <collision>
-            <!--<origin xyz="0 0 0" rpy="0 0 0" />-->
+            <origin xyz="0 0 0" rpy="0 0 0" />
             <geometry>
                 <box size="0.5 0.3 0.07" />

Commit message: ...

File: m2wr_robot/urdf/m2wr.xacro (robot description, xacro)
@@ -2,5 +2,5 @@
 <robot name="m2wr" xmlns:xacro="http://ros.org/wiki/xacro">
     <!-- inludes -->
-    <xacro:include filename="$(find m2wr_robot)/urdf/car_driver.gazebo" />
+    <!--<xacro:include filename="$(find m2wr_robot)/urdf/car_driver.gazebo" />-->
     <xacro:include filename="$(find m2wr_robot)/urdf/wheel.xacro" />
     <xacro:include filename="$(find m2wr_robot)/urdf/caster.xacro" />
@@ -44,3 +44,8 @@
     <xacro:wheel_macro prefix="left_wheel"  parent="base_link" xyz="0  0.1 0.05" r="0.05"/>
     <xacro:wheel_macro prefix="right_wheel" parent="base_link" xyz="0 -0.1 0.05" r="0.05"/>
+    <gazebo>
+        <plugin name="gazebo_ros_control" filename="libgazebo_ros_control.so">
+            <robotNamespace>/m2wr</robotNamespace>
+        </plugin>
+    </gazebo>
 </robot>

File: m2wr_robot/urdf/wheel.xacro (robot description, xacro)
@@ -8,5 +8,17 @@
             <child  link="${prefix}_link"/>
             <axis xyz="0 0 1" />
+            <limit velocity="12.0" effort="0.4" />
+            <dynamics damping="0.1"/>
         </joint>
+        <!-- transimission -->
+        <transmission name="${prefix}_trans" type="SimpleTransmission">
+            <type>transmission_interface/SimpleTransmission</type>
+            <actuator name="${prefix}_motor">
+                <mechanicalReduction>1</mechanicalReduction>
+            </actuator>
+            <joint name="${prefix}_joint">
+                <hardwareInterface>hardware_interface/VelocityJointInterface</hardwareInterface>
+            </joint>
+        </transmission>
         <!-- link -->
         <link name="${prefix}_link">
@@ -29,5 +41,10 @@
         </link>
         <gazebo reference="${prefix}_link">
-          <material>Gazebo/Red</material>
+            <material>Gazebo/Red</material>
+            <material>Gazebo/Red</material>
+            <mu1 value="2.5" />
+            <mu2 value="2.5" />
+            <kp value="50000" />
+            <kd value="10" />
         </gazebo>
     </xacro:macro>

Commit message: ...

File: m2wr_robot/urdf/m2wr.xacro (robot description, xacro)
@@ -1,51 +1,113 @@
 <?xml version="1.0"?>
-<robot name="m2wr" xmlns:xacro="http://ros.org/wiki/xacro">
-    <!-- inludes -->
-    <!--<xacro:include filename="$(find m2wr_robot)/urdf/car_driver.gazebo" />-->
-    <xacro:include filename="$(find m2wr_robot)/urdf/wheel.xacro" />
-    <xacro:include filename="$(find m2wr_robot)/urdf/caster.xacro" />
-    <xacro:include filename="$(find m2wr_robot)/urdf/materials.xacro" />
-    <link name="base_link"/>
-    <!-- body : joint -->
-    <joint name="body_joint" type="fixed">
-        <parent link="base_link"/>
-        <child  link="body_link"/>
-        <origin xyz="-0.07 0 0.07" rpy="0 0 0"/>
+<robot name="dtw_robot" xmlns:xacro="http://ros.org/wiki/xacro">
+  <material name="gray">
+    <color rgba="0.5 0.5 0.5 2.5"/>
+  </material>
+  <material name="red">
+    <color rgba="1.0 0.0 0.0 2.5"/>
+  </material>
+  <xacro:macro name="wheel_macro" params="parent prefix xyz">
+    <joint name="${prefix}_joint" type="continuous">
+      <origin xyz="${xyz}" rpy="${radians(-90)} 0 0"/>
+      <parent link="${parent}"/>
+      <child  link="${prefix}_link"/>
+      <axis xyz="0 0 1" />
     </joint>
-    <!-- body : link -->
-    <link name="body_link">
-        <inertial>
-            <origin xyz="0 0 0" rpy="0 0 0"/>
-            <mass value="1.0"/>
-            <inertia ixx="0.001" ixy="0.0" ixz="0.0" iyy="0.001" iyz="0.0" izz="0.001"/>
-        </inertial>
-        <visual>
-            <origin xyz="0 0 0" rpy="0 0 0" />
-            <geometry>
-                <box size="0.24 0.18 0.06" />
-            </geometry>
-            <material name="gray" />
-        </visual>
-        <collision>
-            <origin xyz="0 0 0" rpy="0 0 0" />
-            <geometry>
-                <box size="0.24 0.178 0.06" />
-            </geometry>
-        </collision>
+    <transmission name="${prefix}_trans" type="SimpleTransmission">
+      <type>transmission_interface/SimpleTransmission</type>
+        <actuator name="${prefix}_motor">
+          <mechanicalReduction>1</mechanicalReduction>
+        </actuator>
+      <joint name="${prefix}_joint">
+        <hardwareInterface>hardware_interface/VelocityJointInterface</hardwareInterface>
+      </joint>
+    </transmission>
+    <link name="${prefix}_link">
+      <inertial>
+        <origin xyz="0 0 0" rpy="0 0 0"/>
+        <mass value="0.1"/>
+        <inertia ixx="0.0001" ixy="0.0" ixz="0.0" iyy="0.0001" iyz="0.0" izz="0.0001"/>
+      </inertial>
+      <visual>
+        <geometry>
+          <cylinder radius="0.05" length="0.02" />
+        </geometry>
+        <material name="red"/>
+      </visual>
+      <collision>
+        <geometry>
+          <cylinder radius="0.05" length="0.02" />
+        </geometry>
+      </collision>
     </link>
-    <gazebo reference="body_link">
-        <material>Gazebo/Gray</material>
+    <gazebo reference="${prefix}_link">
+      <material>Gazebo/Red</material>
+      <mu1 value="2.5" />
+      <mu2 value="2.5" />
+      <kp value="50000" />
+      <kd value="10" />
     </gazebo>
-    <xacro:caster_macro prefix="caster" parent="base_link" xyz="-0.14 0 0.04" r="0.04"/>
-    <!-- front and back caster -->
-    <!--<<xacro:caster_macro prefix="front_caster" parent="base_link" xyz="0.08 0 0.04" r="0.04"/>-->
-    <!--<xacro:caster_macro prefix="back_caster" parent="base_link" xyz="-0.08 0 0.04" r="0.04"/>-->
-    <!-- left and right wheel -->
-    <xacro:wheel_macro prefix="left_wheel"  parent="base_link" xyz="0  0.1 0.05" r="0.05"/>
-    <xacro:wheel_macro prefix="right_wheel" parent="base_link" xyz="0 -0.1 0.05" r="0.05"/>
-    <gazebo>
-        <plugin name="gazebo_ros_control" filename="libgazebo_ros_control.so">
-            <robotNamespace>/m2wr</robotNamespace>
-        </plugin>
-    </gazebo>
+  </xacro:macro>
+  <link name="base_link"/>
+  <joint name="body_joint" type="fixed">
+    <parent link="base_link"/>
+    <child  link="body_link"/>
+    <origin xyz="-0.07 0 0.07" rpy="0 0 0"/>
+  </joint>
+  <link name="body_link">
+    <inertial>
+      <origin xyz="0 0 0" rpy="0 0 0"/>
+      <mass value="1.0"/>
+      <inertia ixx="0.001" ixy="0.0" ixz="0.0" iyy="0.001" iyz="0.0" izz="0.001"/>
+    </inertial>
+    <visual>
+      <origin xyz="0 0 0" rpy="0 0 0" />
+      <geometry>
+        <box size="0.24 0.18 0.06" />
+      </geometry>
+      <material name="gray" />
+    </visual>
+    <collision>
+      <origin xyz="0 0 0" rpy="0 0 0" />
+      <geometry>
+        <box size="0.24 0.178 0.06" />
+      </geometry>
+    </collision>
+  </link>
+  <gazebo reference="body_link">
+    <material>Gazebo/Gray</material>
+  </gazebo>
+  <xacro:wheel_macro prefix="left_wheel"  parent="base_link" xyz="0 0.1 0.05"/>
+  <xacro:wheel_macro prefix="right_wheel" parent="base_link" xyz="0 -0.1 0.05"/>
+  <joint name="ball_joint" type="fixed">
+    <parent link="base_link"/>
+    <child  link="ball_link"/>
+    <origin xyz="-0.14 0 0.04" rpy="0 0 0"/>
+  </joint>
+  <link name="ball_link">
+    <visual>
+      <origin xyz="0 0 0" rpy="0 0 0" />
+      <geometry>
+        <sphere radius="0.04" />
+      </geometry>
+      <material name="gray" />
+    </visual>
+    <collision>
+      <origin xyz="0 0 0" rpy="0 0 0" />
+      <geometry>
+        <sphere radius="0.04" />
+      </geometry>
+      <material name="gray" />
+    </collision>
+  </link>
+  <gazebo reference="ball_link">
+    <material>Gazebo/Gray</material>
+    <mu1 value="0.5" />
+    <mu2 value="0.5" />
+  </gazebo>
+  <gazebo>
+    <plugin name="gazebo_ros_control" filename="libgazebo_ros_control.so">
+      <robotNamespace>/dtw_robot</robotNamespace>
+    </plugin>
+  </gazebo>
 </robot>
