Commit message: ...

File: m2wr_robot/urdf/m2wr.xacro (robot description, xacro)
@@ -1,113 +1,47 @@
 <?xml version="1.0"?>
-<robot name="dtw_robot" xmlns:xacro="http://ros.org/wiki/xacro">
-  <material name="gray">
-    <color rgba="0.5 0.5 0.5 2.5"/>
-  </material>
-  <material name="red">
-    <color rgba="1.0 0.0 0.0 2.5"/>
-  </material>
-  <xacro:macro name="wheel_macro" params="parent prefix xyz">
-    <joint name="${prefix}_joint" type="continuous">
-      <origin xyz="${xyz}" rpy="${radians(-90)} 0 0"/>
-      <parent link="${parent}"/>
-      <child  link="${prefix}_link"/>
-      <axis xyz="0 0 1" />
+<robot name="m2wr" xmlns:xacro="http://ros.org/wiki/xacro">
+    <!-- inludes -->
+    <xacro:include filename="$(find m2wr_robot)/urdf/car_driver.gazebo" />
+    <xacro:include filename="$(find m2wr_robot)/urdf/wheel.xacro" />
+    <xacro:include filename="$(find m2wr_robot)/urdf/caster.xacro" />
+    <xacro:include filename="$(find m2wr_robot)/urdf/materials.xacro" />
+    <link name="base_link"/>
+    <!-- body : joint -->
+    <joint name="body_joint" type="fixed">
+        <parent link="base_link"/>
+        <child  link="body_link"/>
+        <origin xyz="0 0 0.07" rpy="0 0 0"/>
     </joint>
-    <transmission name="${prefix}_trans" type="SimpleTransmission">
-      <type>transmission_interface/SimpleTransmission</type>
-        <actuator name="${prefix}_motor">
-          <mechanicalReduction>1</mechanicalReduction>
-        </actuator>
-      <joint name="${prefix}_joint">
-        <hardwareInterface>hardware_interface/VelocityJointInterface</hardwareInterface>
-      </joint>
-    </transmission>
-    <link name="${prefix}_link">
-      <inertial>
-        <origin xyz="0 0 0" rpy="0 0 0"/>
-        <mass value="0.1"/>
-        <inertia ixx="0.0001" ixy="0.0" ixz="0.0" iyy="0.0001" iyz="0.0" izz="0.0001"/>
-      </inertial>
-      <visual>
-        <geometry>
-          <cylinder radius="0.05" length="0.02" />
-        </geometry>
-        <material name="red"/>
-      </visual>
-      <collision>
-        <geometry>
-          <cylinder radius="0.05" length="0.02" />
-        </geometry>
-      </collision>
+    <!-- body : link -->
+    <link name="body_link">
+        <inertial>
+            <origin xyz="0 0 0" rpy="0 0 0"/>
+            <mass value="1.0"/>
+            <inertia ixx="0.001" ixy="0.0" ixz="0.0" iyy="0.001" iyz="0.0" izz="0.001"/>
+        </inertial>
+        <visual>
+            <origin xyz="0 0 0" rpy="0 0 0" />
+            <geometry>
+                <box size="0.24 0.18 0.06" />
+            </geometry>
+            <material name="gray" />
+        </visual>
+        <collision>
+            <origin xyz="0 0 0" rpy="0 0 0" />
+            <geometry>
+                <box size="0.24 0.178 0.06" />
+            </geometry>
+        </collision>
     </link>
-    <gazebo reference="${prefix}_link">
-      <material>Gazebo/Red</material>
-      <mu1 value="2.5" />
-      <mu2 value="2.5" />
-      <kp value="50000" />
-      <kd value="10" />
+    <gazebo reference="body_link">
+        <material>Gazebo/Gray</material>
     </gazebo>
-  </xacro:macro>
-  <link name="base_link"/>
-  <joint name="body_joint" type="fixed">
-    <parent link="base_link"/>
-    <child  link="body_link"/>
-    <origin xyz="-0.07 0 0.07" rpy="0 0 0"/>
-  </joint>
-  <link name="body_link">
-    <inertial>
-      <origin xyz="0 0 0" rpy="0 0 0"/>
-      <mass value="1.0"/>
-      <inertia ixx="0.001" ixy="0.0" ixz="0.0" iyy="0.001" iyz="0.0" izz="0.001"/>
-    </inertial>
-    <visual>
-      <origin xyz="0 0 0" rpy="0 0 0" />
-      <geometry>
-        <box size="0.24 0.18 0.06" />
-      </geometry>
-      <material name="gray" />
-    </visual>
-    <collision>
-      <origin xyz="0 0 0" rpy="0 0 0" />
-      <geometry>
-        <box size="0.24 0.178 0.06" />
-      </geometry>
-    </collision>
-  </link>
-  <gazebo reference="body_link">
-    <material>Gazebo/Gray</material>
-  </gazebo>
-  <xacro:wheel_macro prefix="left_wheel"  parent="base_link" xyz="0 0.1 0.05"/>
-  <xacro:wheel_macro prefix="right_wheel" parent="base_link" xyz="0 -0.1 0.05"/>
-  <joint name="ball_joint" type="fixed">
-    <parent link="base_link"/>
-    <child  link="ball_link"/>
-    <origin xyz="-0.14 0 0.04" rpy="0 0 0"/>
-  </joint>
-  <link name="ball_link">
-    <visual>
-      <origin xyz="0 0 0" rpy="0 0 0" />
-      <geometry>
-        <sphere radius="0.04" />
-      </geometry>
-      <material name="gray" />
-    </visual>
-    <collision>
-      <origin xyz="0 0 0" rpy="0 0 0" />
-      <geometry>
-        <sphere radius="0.04" />
-      </geometry>
-      <material name="gray" />
-    </collision>
-  </link>
-  <gazebo reference="ball_link">
-    <material>Gazebo/Gray</material>
-    <mu1 value="0.5" />
-    <mu2 value="0.5" />
-  </gazebo>
-  <gazebo>
-    <plugin name="gazebo_ros_control" filename="libgazebo_ros_control.so">
-      <robotNamespace>/dtw_robot</robotNamespace>
-    </plugin>
-  </gazebo>
+    <!-- front and back caster -->
+    <xacro:caster_macro prefix="back_caster" parent="base_link" xyz="-0.08 0 0.04" r="0.04"/>
+    <xacro:caster_macro prefix="front_caster" parent="base_link" xyz="0.08 0 0.04" r="0.04"/>
+    <!-- left and right wheel -->
+    <xacro:wheel_macro prefix="left_wheel"  parent="base_link" xyz="0  0.1 0.05" r="0.05"/>
+    <xacro:wheel_macro prefix="right_wheel" parent="base_link" xyz="0 -0.1 0.05" r="0.05"/>
+    <!-- driver for two wheel car -->
+    <xacro:car_driver_micro pubTopic="/cmd_vel" odomTopic="/odom"/>
 </robot>

Commit message: ...

File: m2wr_robot/urdf/m2wr.xacro (robot description, xacro)
@@ -45,4 +45,4 @@
     <xacro:wheel_macro prefix="right_wheel" parent="base_link" xyz="0 -0.1 0.05" r="0.05"/>
     <!-- sensor -->
-    <xacro:lidar_macro prefix="lidar" parent="base_link" xyz="0 0 0.15" r="0.05" l="0.10" model="m2wr"/>
+    <xacro:lidar_macro prefix="lidar" parent="base_link" xyz="0 0 0.15" r="0.05" l="0.10"/>
 </robot>

File: m2wr_robot/urdf/sensor/lidar.xacro (robot description, xacro)
@@ -1,5 +1,5 @@
 <?xml version="1.0"?>
 <robot xmlns:xacro="http://ros.org/wiki/xacro">
-    <xacro:macro name="lidar_macro" params="parent prefix xyz r l model">
+    <xacro:macro name="lidar_macro" params="parent prefix xyz r l">
         <joint name="${prefix}_joint" type="fixed">
             <parent link="${parent}"/>
@@ -48,5 +48,5 @@
             </ray>
             <plugin name="gazebo_ros_head_hokuyo_controller" filename="libgazebo_ros_laser.so">
-                <topicName value="${model}/laser/scan" />
+                <topicName>/m2wr/laser/scan</topicName>
                 <frameName>sensor_laser</frameName>
             </plugin>

Commit message: ...

File: m2wr_robot/urdf/m2wr.xacro (robot description, xacro)
@@ -45,4 +45,4 @@
     <xacro:wheel_macro prefix="right_wheel" parent="base_link" xyz="0 -0.1 0.05" r="0.05"/>
     <!-- sensor -->
-    <xacro:lidar_macro prefix="lidar" parent="base_link" xyz="0 0 0.15" r="0.05" l="0.10"/>
+    <xacro:lidar_macro prefix="lidar" parent="base_link" xyz="0 0 0.15" r="0.05" l="0.10" model="m2wr"/>
 </robot>

File: m2wr_robot/urdf/sensor/lidar.xacro (robot description, xacro)
@@ -1,5 +1,5 @@
 <?xml version="1.0"?>
 <robot xmlns:xacro="http://ros.org/wiki/xacro">
-    <xacro:macro name="lidar_macro" params="parent prefix xyz r l">
+    <xacro:macro name="lidar_macro" params="parent prefix xyz r l model">
         <joint name="${prefix}_joint" type="fixed">
             <parent link="${parent}"/>
@@ -48,5 +48,5 @@
                 </ray>
                 <plugin name="gazebo_ros_head_hokuyo_controller" filename="libgazebo_ros_laser.so">
-                    <topicName>/m2wr/laser/scan</topicName>
+                    <topicName value="${model}/laser/scan" />
                     <frameName>sensor_laser</frameName>
                 </plugin>

Commit message: ...

File: m2wr_robot/urdf/m2wr.xacro (robot description, xacro)
@@ -6,5 +6,6 @@
     <xacro:include filename="$(find m2wr_robot)/urdf/caster.xacro" />
     <xacro:include filename="$(find m2wr_robot)/urdf/materials.xacro" />
-    <xacro:include filename="$(find m2wr_robot)/urdf/sensor/lidar.xacro" />
+    <!--<xacro:include filename="$(find m2wr_robot)/urdf/sensor/lidar.xacro" />-->
+    <xacro:include filename="$(find m2wr_robot)/urdf/sensor/camera.xacro" />
     <link name="base_link"/>
     <!-- body : joint -->
@@ -31,5 +32,5 @@
             <origin xyz="0 0 0" rpy="0 0 0" />
             <geometry>
-                <box size="0.24 0.178 0.06" />
+                <box size="0.24 0.18 0.06" />
             </geometry>
         </collision>
@@ -45,5 +46,7 @@
     <xacro:wheel_macro prefix="right_wheel" parent="base_link" xyz="0 -0.1 0.05" r="0.05"/>
     <!-- sensor -->
-    <xacro:include filename="$(find m2wr_robot)/urdf/sensor/lidar.gazebo" />
-    <xacro:lidar_macro prefix="lidar" parent="base_link" xyz="0 0 0.15" r="0.05" l="0.10"/>
+    <!--<xacro:include filename="$(find m2wr_robot)/urdf/sensor/lidar.gazebo" />-->
+    <!--<xacro:lidar_macro prefix="lidar" parent="base_link" xyz="0 0 0.15" r="0.05" l="0.10"/>-->
+    <xacro:include filename="$(find m2wr_robot)/urdf/sensor/camera.gazebo" />
+    <xacro:camera_macro prefix="camera" parent="base_link" xyz="0.11 0 0.15" Sxyz="0.02, 0.06, 0.04"/>
 </robot>

Commit message: ...

File: m2wr_robot/urdf/m2wr.xacro (robot description, xacro)
@@ -49,4 +49,4 @@
     <!--<xacro:lidar_macro prefix="lidar" parent="base_link" xyz="0 0 0.15" r="0.05" l="0.10"/>-->
     <!--<xacro:include filename="$(find m2wr_robot)/urdf/sensor/camera.gazebo" />-->
-    <xacro:camera_macro prefix="camera" parent="base_link" xyz="0.11 0 0.15" Sxyz="0.02, 0.06, 0.04"/>
+    <xacro:camera_macro prefix="camera" parent="base_link" xyz="0.11 0 0.16" Sxyz="0.02, 0.06, 0.04"/>
 </robot>

File: m2wr_robot/urdf/sensor/camera.xacro (robot description, xacro)
@@ -7,5 +7,5 @@
             <visual>
                 <geometry>
-                    <box size="Sxyz"/>
+                    <box size="${Sxyz}"/>
                 </geometry>
             <material name="white"/>
