Commit message: ...

File: m2wr_robot/urdf/sensor/lidar.xacro (robot description, xacro)
@@ -1,5 +1,5 @@
 <?xml version="1.0"?>
 <robot xmlns:xacro="http://ros.org/wiki/xacro">
-    <xacro:macro name="lidar_macro" params="parent prefix xyz r l model">
+    <xacro:macro name="lidar_macro" params="parent prefix xyz r l">
         <joint name="${prefix}_joint" type="fixed">
             <parent link="${parent}"/>
@@ -48,5 +48,5 @@
                 </ray>
                 <plugin name="gazebo_ros_head_hokuyo_controller" filename="libgazebo_ros_laser.so">
-                    <topicName value="${model}/laser/scan" />
+                    <topicName>m2wr/laser/scan</topicName>
                     <frameName>sensor_laser</frameName>
                 </plugin>
