Commit message: ...

File: m2wr_robot/urdf/sensor/camera.xacro (robot description, xacro)
@@ -2,25 +2,26 @@
 <robot xmlns:xacro="http://ros.org/wiki/xacro">
     <xacro:macro name="camera_macro" params="parent prefix xyz Sxyz">
-    <!-- sensor : link -->
-    <link name="%{prefix}_link">
-        <!-- visual -->
-        <visual>
-            <geometry>
-                <box size="Sxyz"/>
-            </geometry>
-        <material name="white"/>
-        </visual>
-        <!-- collsion -->
-        <collision>
-            <geometry>
-                <box size="Sxyz"/>
-            </geometry>
-        </collision>
-    </link>
-    <!-- sensor : joint -->
-    <joint name="${prefix}_joint" type="fixed">
-        <origin xyz="${xyz}" rpy="0 0 0"/>
-        <parent link="${parent}"/>
-        <child link="${prefix}_link"/>
-    </joint>
+        <!-- sensor : link -->
+        <link name="%{prefix}_link">
+            <!-- visual -->
+            <visual>
+                <geometry>
+                    <box size="Sxyz"/>
+                </geometry>
+            <material name="white"/>
+            </visual>
+            <!-- collsion -->
+            <collision>
+                <geometry>
+                    <box size="Sxyz"/>
+                </geometry>
+            </collision>
+        </link>
+        <!-- sensor : joint -->
+        <joint name="${prefix}_joint" type="fixed">
+            <origin xyz="${xyz}" rpy="0 0 0"/>
+            <parent link="${parent}"/>
+            <child link="${prefix}_link"/>
+        </joint>
+    </xacro:macro>
 </robot>

Commit message: ...

File: m2wr_robot/urdf/sensor/camera.xacro (robot description, xacro)
@@ -3,5 +3,5 @@
     <xacro:macro name="camera_macro" params="parent prefix xyz Sxyz">
         <!-- sensor : link -->
-        <link name="%{prefix}_link">
+        <link name="${prefix}_link">
             <!-- visual -->
             <visual>

Commit message: ...

File: m2wr_robot/urdf/sensor/camera.xacro (robot description, xacro)
@@ -14,5 +14,5 @@
             <collision>
                 <geometry>
-                    <box size="Sxyz"/>
+                    <box size="${Sxyz}"/>
                 </geometry>
             </collision>
